File: board/camera_trigger.kicad_pcb (KiCad board)
At the start: 2 copper layers, 36 x 100 mm, 40 parts, among them J1 LIDAR, J2 Rotary switch, J3 PowerBoost 1000C, J4 Display, J5 Audio-Jack-3, Q1 Q_NPN_BEC, Q2 Q_NPN_BEC, Q3 Q_NPN_BEC, Q4 Q_NPN_BEC, U1 OPA340UA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

Commit message: Added OSHW logo
Parts:
- added REF**: OSHW-Logo_5.7x6mm_SilkScreen, Symbol:OSHW-Logo_5.7x6mm_SilkScreen, F.Cu at (83.8, 53.3)
